Commit message: Update T3 URDF and mesh assets

File: ardy/retarget_to_t3/assets/t3_robot/T3.urdf (robot description, URDF)
Before this commit: robot T3, 36 links, 35 joints
Joints:
- joint head_pitch_joint: origin xyz=-0.00011475 0.020709 0.42181 rpy=0 0 0 -> xyz=-0.00011475 0 0.395710 rpy=0 0 0
- joint head_yaw_joint: origin xyz=0 -0.0189 0.1325 rpy=0 0 0 -> xyz=0 0 0.033976 rpy=0 0 0
- joint waist_pitch_joint: origin xyz=0 0 0 rpy=0 0 0 -> xyz=0.005236 0 0 rpy=0 0 0

Commit message: Align Nero shoulders with trunk panels

File: ardy/retarget_to_t3/assets/t3_robot/T3.urdf (robot description, URDF)
Before this commit: robot T3, 36 links, 35 joints
Joints:
- joint torso_to_left_nero_base: origin xyz=0.00197790 0.07684000 0.35792000 rpy=1.5707963267948966 -1.5707963267948966 3.141592653589793 -> xyz=0.00197790 0.07684000 0.32038000 rpy=1.5707963267948966 -1.5707963267948966 3.141592653589793
- joint torso_to_right_nero_base: origin xyz=0.00197060 -0.07316000 0.35789000 rpy=1.5707963267948966 -1.5707963267948966 0 -> xyz=0.00197060 -0.07316000 0.32038000 rpy=1.5707963267948966 -1.5707963267948966 0

Commit message: Replace T3 base and wheel assets

File: ardy/retarget_to_t3/assets/t3_robot/T3.urdf (robot description, URDF)
Before this commit: robot T3, 36 links, 35 joints
Links:
- link base_link: geometry collision box size=0.5464 0.23 0.1806; visual mesh filename=meshes/wheel_base/base.stl
- link left_wheel_link: geometry collision cylinder length=0.1048 radius=0.10; visual mesh filename=meshes/wheel_base/wheels.stl
- link right_wheel_link: geometry collision cylinder length=0.1048 radius=0.10; visual mesh filename=meshes/wheel_base/wheels.stl
Joints:
- joint left_wheel_joint: origin xyz=0 0.19 0.10 rpy=0 0 0 -> xyz=0 0.1678 0.09999 rpy=0 0 0
- joint right_wheel_joint: origin xyz=0 -0.19 0.10 rpy=0 0 0 -> xyz=0 -0.1678 0.09999 rpy=0 0 0
